File: COMET1_PWR_Board/COMET1_PWR_Board.kicad_sch (KiCad schematic)
At the start: 0 parts

Commit message: PCBs Update - Near Complete
Other:
- sheet Block Diagram: file Block Diagram.kicad_sch -> SubSchematics/Block Diagram.kicad_sch
- sheet Component Specs: file Component Specs.kicad_sch -> SubSchematics/Component Specs.kicad_sch
- sheet Power Board Schematic: file PowerBoard.kicad_sch -> SubSchematics/PowerBoard.kicad_sch
Changed lines of the file:
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@@
 	(title_block
 		(title "Cover Page")
-		(date "Last Modified Date")
+		(date "2025-12-23")
 		(rev "${REVISION}")
 		(company "${COMPANY}")
@@
 			(type dot)
 			(color 0 0 0 1)
+		)
+	)
+	(sheet
+		(at 342.9 302.26)
+		(size 35.56 5.08)
+		(exclude_from_sim no)
+		(in_bom yes)
+		(on_board yes)
+		(dnp no)
+		(stroke
+			(width 0.1524)
+			(type solid)
+		)
+		(fill
+			(color 0 0 0 0.0000)
+		)
+		(property "Sheetname" "Component Specs"
+			(at 342.9 301.2309 0)
+			(effects
+				(font
+					(face "Times New Roman")
+					(size 1.905 1.905)
+					(bold yes)
+					(color 0 0 0 1)
+				)
+				(justify left bottom)
+			)
+		)
+		(property "Sheetfile" "SubSchematics/Component Specs.kicad_sch"
+			(at 344.17 303.53 0)
+			(effects
+				(font
+					(face "Arial")
+					(size 1.27 1.27)
+				)
+				(justify left top)
+			)
+		)
+		(instances
+			(project "COMET1_PWR_Board"
+				(path "/0650c7a8-acba-429c-9f8e-eec0baf0bc1c"
+					(page "4")
+				)
+			)
 		)
 	)
@@
 			)
 		)
-		(property "Sheetfile" "Block Diagram.kicad_sch"
+		(property "Sheetfile" "SubSchematics/Block Diagram.kicad_sch"
 			(at 300.99 303.53 0)
 			(effects
@@
 				(path "/0650c7a8-acba-429c-9f8e-eec0baf0bc1c"
 					(page "2")
-				)
-			)
-		)
-	)
-	(sheet
-		(at 339.09 302.26)
-		(size 33.02 5.08)
-		(exclude_from_sim no)
-		(in_bom yes)
-		(on_board yes)
-		(dnp no)
-		(fields_autoplaced yes)
-		(stroke
-			(width 0.1524)
-			(type solid)
-		)
-		(fill
-			(color 0 0 0 0.0000)
-		)
-		(property "Sheetname" "Component Specs"
-			(at 339.09 301.5484 0)
-			(effects
-				(font
-					(size 1.27 1.27)
-				)
-				(justify left bottom)
-			)
-		)
-		(property "Sheetfile" "Component Specs.kicad_sch"
-			(at 339.09 307.9246 0)
-			(effects
-				(font
-					(size 1.27 1.27)
-				)
-				(justify left top)
-			)
-		)
-		(instances
-			(project "COMET1_PWR_Board"
-				(path "/0650c7a8-acba-429c-9f8e-eec0baf0bc1c"
-					(page "4")
 				)
 			)
@@
 			)
 		)
-		(property "Sheetfile" "PowerBoard.kicad_sch"
+		(property "Sheetfile" "SubSchematics/PowerBoard.kicad_sch"
 			(at 300.99 314.96 0)
 			(effects
