File: COMET1_CCT_Board/COMET1_CCT.kicad_sch (KiCad schematic)
At the start: 0 parts

Commit message: PCBs Update - Near Complete
Other:
- sheet Block Diagram: file Block Diagram.kicad_sch -> SubSchematics/Block Diagram.kicad_sch
- sheet CCT Board Schematic: file CCT Board Schematic.kicad_sch -> SubSchematics/CCT Board Schematic.kicad_sch
- note added: "CCT Board Schematic"
- note added: "MCU & Peripherals"
- note added: "RS485"
- note added: "Sensors"
- note added: "USBC"
- note removed: "Power - Sequencing"
- note removed: "Project Architecture"
- note removed: "Random Sheet 1"
- note removed: "Random Sheet 2"
- note removed: "Revision History"

Commit message: PCBs update - Near Complete x2
Other:
- note added: "ADD FUNCTIONALITY FOR EXTERNAL WARNING LIGHT AT ROCKET FOR ARMING AND COUNTDOWN"
Changed lines of the file:
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@@
+		)
+	)
+	(text "ADD FUNCTIONALITY FOR EXTERNAL WARNING LIGHT AT ROCKET\nFOR ARMING AND COUNTDOWN"
+		(exclude_from_sim no)
+		(at 203 105 0)
+		(effects
+			(font
+				(face "Times New Roman")
+				(size 8 8)
+				(thickness 0.6)
+				(bold yes)
+				(color 0 0 255 1)
+			)
+			(justify bottom)
 		)
 	)

Commit message: kicad files changes
Other:
- note added: "ADD FUNCTIONALITY FOR EXTERNAL WARNING LIGHT AT ROCKET FOR ARMING AND COUNTDOWN PCB STITCHING VIAS PCB VCUTS/PANEL? + TOOLING HOLES"
- note removed: "ADD FUNCTIONALITY FOR EXTERNAL WARNING LIGHT AT ROCKET FOR ARMING AND COUNTDOWN"
Changed lines of the file:
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@@
 		)
 	)
-	(text "ADD FUNCTIONALITY FOR EXTERNAL WARNING LIGHT AT ROCKET\nFOR ARMING AND COUNTDOWN"
+	(text "ADD FUNCTIONALITY FOR EXTERNAL WARNING LIGHT AT ROCKET\nFOR ARMING AND COUNTDOWN\n\nPCB STITCHING VIAS\n\nPCB VCUTS/PANEL? + TOOLING HOLES"
 		(exclude_from_sim no)
-		(at 203 105 0)
+		(at 205.4 167.2 0)
 		(effects
 			(font
