File: COMET1_CCT_Board/SubSchematics/Block Diagram.kicad_sch (KiCad schematic)
At the start: 0 parts

Commit message: PCBs update - Near Complete x2
Changed lines of the file:
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@@
 		)
 	)
-	(text_box "GPIO_??"
+	(text_box "GPIO_36"
 		(exclude_from_sim no)
 		(at 264 214.5 0)
@@
 		)
 	)
-	(text_box "A: I2C_0x??\nB: I2C_0x??"
+	(text_box "A: I2C_0x6E\nB: I2C_0x60"
 		(exclude_from_sim no)
 		(at 264 92 0)
@@
 		)
 	)
-	(text_box "Ext. Thermocouple Interface"
+	(text_box "Ext. Thermocouple ADC"
 		(exclude_from_sim no)
 		(at 329 175 0)
@@
 		)
 	)
-	(text_box "FILL - GPIO_??\nARM - GPIO_??\nFIRE - GPIO_??\n"
+	(text_box "FIRE - GPIO_4\nARM - GPIO_5\nFILL - GPIO_6\n\n"
 		(exclude_from_sim no)
 		(at 187 190.758 0)
@@
 		)
 	)
-	(text_box "GPIO_??\nGPIO_??"
+	(text_box "Red - GPIO_38\nGreen - GPIO_39"
 		(exclude_from_sim no)
 		(at 264 202.5 0)
 		(size 18.088 7)
-		(margins 1.7144 1.7144 1.7144 1.7144)
+		(margins 1 1 1 1)
 		(stroke
 			(width -0.0001)
@@
 			(font
 				(face "Times New Roman")
-				(size 2.286 2.286)
+				(size 1.5 1.5)
 				(italic yes)
 				(color 162 22 34 1)
@@
 		)
 	)
-	(text_box "RED LED\nGREEN LED"
+	(text_box "STATUS LEDs"
 		(exclude_from_sim no)
 		(at 284 201.5 0)
@@
 		(fill
 			(type color)
-			(color 175 67 103 1)
+			(color 194 117 135 1)
 		)
 		(effects
@@
 		)
 	)
-	(text_box "GPIO_??"
+	(text_box "GPIO_13"
 		(exclude_from_sim no)
 		(at 187 73 0)
@@
 		(fill
 			(type color)
-			(color 175 67 103 1)
+			(color 194 117 135 1)
 		)
 		(effects
@@
 		)
 	)
-	(text_box "Addr. = 0x??"
+	(text_box "Addr. = 0x44"
 		(exclude_from_sim no)
 		(at 264 102 0)
@@
 		)
 	)
-	(text_box "Addr. = 0x??"
+	(text_box "Addr. = 0x20"
 		(exclude_from_sim no)
 		(at 264 125 0)
@@
 		(fill
 			(type color)
-			(color 175 67 103 1)
-		)
-		(effects
+			(color 194 117 135 1)
+		)
+		(effects
