File: COMET1_CCT_Board/SubSchematics/CCT Board Schematic.kicad_sch (KiCad schematic)
At the start: 9 parts, among them J1 DF11-10DS-2DSA, J2 DF11-10DS-2DSA

Commit message: PCBs update - Near Complete x2
Parts:
- FID1, FID2, FID3: symbol 0_Peripherals:Fiducial -> 0_Mechanical:Fiducial
- J1, J2: Farnell Link https://uk.farnell.com/hirose-hrs/df11-10ds-2dsa-05/recepta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 -> (none); Farnell Part Number 1688320 -> (none); Farnell Price 1.4 -> (none); JLC Part Number C5712177 -> (none); JLC Price 0.89 -> (none); Min Qty (none) -> 1; Order Code (none) -> 1688320; Part Link (none) -> https://uk.farnell.com/hirose-hrs/df11-10ds-2dsa-05/recepta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; Price Per (none) -> 1.4; Supplier (none) -> Farnell
- MH1, MH2, MH3, MH4: symbol 0_Peripherals:MountingHole_Pad -> 0_Mechanical:MountingHole_Pad
Changed lines of the file:
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@@
 	)
 	(symbol
-		(lib_id "0_Peripherals:MountingHole_Pad")
+		(lib_id "0_Mechanical:MountingHole_Pad")
 		(at 132.08 214.63 0)
 		(unit 1)
@@
 			)
 		)
-		(property "JLC Part Number" ""
-			(at 132.08 214.63 0)
-			(effects
-				(font
-					(size 1.27 1.27)
-				)
-				(hide yes)
-			)
-		)
-		(property "JLC Price" ""
-			(at 132.08 214.63 0)
-			(effects
-				(font
-					(size 1.27 1.27)
-				)
-				(hide yes)
-			)
-		)
 		(pin "1"
 		)
@@
 	)
 	(symbol
-		(lib_id "0_Peripherals:Fiducial")
+		(lib_id "0_Mechanical:Fiducial")
 		(at 161.29 218.44 0)
 		(mirror y)
@@
 			)
 		)
-		(property "JLC Part Number" ""
-			(at 161.29 218.44 0)
-			(effects
-				(font
-					(size 1.27 1.27)
-				)
-				(hide yes)
-			)
-		)
-		(property "JLC Price" ""
-			(at 161.29 218.44 0)
-			(effects
-				(font
-					(size 1.27 1.27)
-				)
-				(hide yes)
-			)
-		)
 		(instances
 			(project "COMET1_CCT"
@@
 	)
 	(symbol
-		(lib_id "0_Peripherals:MountingHole_Pad")
+		(lib_id "0_Mechanical:MountingHole_Pad")
 		(at 139.7 214.63 0)
 		(unit 1)
@@
 			)
 		)
-		(property "JLC Part Number" ""
-			(at 139.7 214.63 0)
-			(effects
-				(font
-					(size 1.27 1.27)
-				)
-				(hide yes)
-			)
-		)
-		(property "JLC Price" ""
-			(at 139.7 214.63 0)
-			(effects
-				(font
-					(size 1.27 1.27)
-				)
-				(hide yes)
-			)
-		)
 		(pin "1"
 		)
@@
 	)
 	(symbol
-		(lib_id "0_Peripherals:Fiducial")
+		(lib_id "0_Mechanical:Fiducial")
 		(at 161.29 210.82 0)
 		(mirror y)
@@
 			)
 		)
-		(property "JLC Part Number" ""
-			(at 161.29 210.82 0)
-			(effects
-				(font
-					(size 1.27 1.27)
-				)
-				(hide yes)
-			)
-		)
-		(property "JLC Price" ""
-			(at 161.29 210.82 0)
-			(effects
-				(font
-					(size 1.27 1.27)
-				)
-				(hide yes)
-			)
-		)
 		(instances
 			(project "COMET1_CCT"
@@
 	)
 	(symbol
-		(lib_id "Library:GND")
+		(lib_id "power:GND")
 		(at 261.62 173.99 0)
 		(unit 1)
@@
 	)
 	(symbol
-		(lib_id "Library:GND")
+		(lib_id "power:GND")
 		(at 261.62 121.92 0)
 		(unit 1)
@@
 	)
 	(symbol
-		(lib_id "0_Peripherals:Fiducial")
+		(lib_id "0_Mechanical:Fiducial")
 		(at 161.29 214.63 0)
 		(mirror y)
@@
 			)
 		)
-		(property "JLC Part Number" ""
-			(at 161.29 214.63 0)
-			(effects
-				(font
-					(size 1.27 1.27)
-				)
-				(hide yes)
-			)
-		)
-		(property "JLC Price" ""
-			(at 161.29 214.63 0)
-			(effects
-				(font
-					(size 1.27 1.27)
-				)
-				(hide yes)
-			)
-		)
 		(instances
 			(project "COMET1_CCT"
@@
 	)
 	(symbol
-		(lib_id "0_Peripherals:MountingHole_Pad")
+		(lib_id "0_Mechanical:MountingHole_Pad")
 		(at 116.84 214.63 0)
 		(unit 1)
@@
 			)
 		)
-		(property "JLC Part Number" ""
-			(at 116.84 214.63 0)
-			(effects
-				(font
-					(size 1.27 1.27)
-				)
-				(hide yes)
-			)
-		)
-		(property "JLC Price" ""
-			(at 116.84 214.63 0)
-			(effects
-				(font
-					(size 1.27 1.27)
-				)
-				(hide yes)
-			)
-		)
 		(pin "1"
 		)
@@
 	)
 	(symbol
-		(lib_id "0_Peripherals:MountingHole_Pad")
+		(lib_id "0_Mechanical:MountingHole_Pad")
 		(at 124.46 214.63 0)
 		(unit 1)
@@
 		)
 		(property "Description" "Mounting Hole with connection"
-			(at 124.46 214.63 0)
-			(effects
-				(font
-					(size 1.27 1.27)
-				)
-				(hide yes)
-			)
-		)
-		(property "JLC Part Number" ""
-			(at 124.46 214.63 0)
-			(effects
-				(font
-					(size 1.27 1.27)
-				)
-				(hide yes)
-			)
-		)
-		(property "JLC Price" ""
 			(at 124.46 214.63 0)
 			(effects
@@
 			)
 		)
-		(property "JLC Part Number" "C5712177"
-			(at 264.16 118.11 0)
-			(effects
-				(font
-					(size 1.27 1.27)
-				)
-				(hide yes)
-			)
-		)
-		(property "JLC Price" "0.89"
-			(at 264.16 118.11 0)
-			(effects
-				(font
-					(size 1.27 1.27)
-				)
-				(hide yes)
-			)
-		)
 		(property "MPN" "DF11-10DS-2DSA"
 			(at 264.16 118.11 0)
@@
 			)
 		)
-		(property "Farnell Link" "https://uk.farnell.com/hirose-hrs/df11-10ds-2dsa-05/receptacle-2mm-10way/dp/1688320"
+		(property "Min Qty" "1"
 			(at 264.16 118.11 0)
 			(effects
@@
 			)
 		)
-		(property "Farnell Part Number" "1688320"
+		(property "Order Code" "1688320"
 			(at 264.16 118.11 0)
 			(effects
@@
 			)
 		)
-		(property "Farnell Price" "1.4"
+		(property "Part Link" "https://uk.farnell.com/hirose-hrs/df11-10ds-2dsa-05/receptacle-2mm-10way/dp/1688320"
 			(at 264.16 118.11 0)
 			(effects
@@
 			)
 		)
+		(property "Price Per" "1.4"
+			(at 264.16 118.11 0)
+			(effects
+				(font
+					(size 1.27 1.27)
+				)
+				(hide yes)
+			)
+		)
+		(property "Supplier" "Farnell"
+			(at 264.16 118.11 0)
+			(effects
+				(font
+					(size 1.27 1.27)
+				)
+				(hide yes)
+			)
+		)
 		(pin "5"
 		)
@@
 	)
 	(symbol
-		(lib_id "Library:+3V3")
+		(lib_id "power:+3V3")
 		(at 261.62 92.71 0)
 		(unit 1)
@@
 	)
 	(symbol
-		(lib_id "Library:+3V3")
+		(lib_id "power:+3V3")
 		(at 261.62 144.78 0)
 		(unit 1)
@@
 			)
 		)
-		(property "JLC Part Number" "C5712177"
-			(at 264.16 147.32 0)
-			(effects
-				(font
-					(size 1.27 1.27)
-				)
-				(hide yes)
-			)
-		)
-		(property "JLC Price" "0.89"
-			(at 264.16 147.32 0)
-			(effects
-				(font
-					(size 1.27 1.27)
-				)
-				(hide yes)
-			)
-		)
 		(property "MPN" "DF11-10DS-2DSA"
 			(at 264.16 147.32 0)
@@
 			)
 		)
-		(property "Farnell Link" "https://uk.farnell.com/hirose-hrs/df11-10ds-2dsa-05/receptacle-2mm-10way/dp/1688320"
+		(property "Min Qty" "1"
 			(at 264.16 147.32 0)
 			(effects
@@
 			)
 		)
-		(property "Farnell Part Number" "1688320"
+		(property "Order Code" "1688320"
 			(at 264.16 147.32 0)
 			(effects
@@
 			)
 		)
-		(property "Farnell Price" "1.4"
+		(property "Part Link" "https://uk.farnell.com/hirose-hrs/df11-10ds-2dsa-05/receptacle-2mm-10way/dp/1688320"
 			(at 264.16 147.32 0)
 			(effects
+				(font
+					(size 1.27 1.27)
+				)
+				(hide yes)
+			)
+		)
+		(property "Price Per" "1.4"
+			(at 264.16 147.32 0)
+			(effects
+				(font
+					(size 1.27 1.27)
+				)
+				(hide yes)
+			)
+		)
+		(property "Supplier" "Farnell"
+			(at 264.16 147.32 0)
+			(effects
