File: COMET1_CCT_Board/SubSchematics/MCU & Peripherals.kicad_sch (KiCad schematic)
At the start: 41 parts, among them J12 Molex_01x02, J13 Conn_02x03_Odd_Even, J3 Micro_SD_Card, J4 Pin_01x02, U1 RP2350_80QFN, U2 S25FL128, X1 ABM8-272-T3

Commit message: PCBs Update - Near Complete
Parts:
- BUZ1: JLC Part Number (none) -> C95299; JLC Price (none) -> 0.17; MPN (none) -> MLT-7525
- C1, C15, C2, C3: JLC Part Number (none) -> C23733; JLC Price (none) -> 0.0035; MPN (none) -> CL05A475MP5NRNC
- C10, C11, C12, C13, C14, C4, C5, C6, C7, C8, C9: JLC Part Number (none) -> C1525; JLC Price (none) -> 0.0009; MPN (none) -> CL05B104KO5NNNC
- C16, C17: JLC Part Number (none) -> C1548; JLC Price (none) -> 0.0007; MPN (none) -> 0402CG150J500NT
- C18, C19: JLC Part Number (none) -> C14663; JLC Price (none) -> 0.002; MPN (none) -> CC0603KRX7R9BB104
- D1: footprint 0_Passives:LED_0805_2012Metric -> 0_Passives:D_SOD-323; JLC Part Number (none) -> C2128; JLC Price (none) -> 0.0064; MPN (none) -> 1N4148WS
- J12: Farnell Link (none) -> https://uk.farnell.com/molex/502352-0201/wtb-conn-header-2p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; Farnell Part Number (none) -> 3103081; Farnell Price (none) -> 0.95; JLC Part Number (none) -> C587898; JLC Price (none) -> 0.22; Supplier Link https://uk.farnell.com/molex/502352-0201/wtb-conn-header-2p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 -> (none)
- J13: value Conn_02x03_Odd_Even -> Conn_02x03; JLC Part Number (none) -> N/A; JLC Price (none) -> N/A; MPN (none) -> N/A; now not fitted
- J3: Farnell Link (none) -> https://uk.farnell.com/molex/47219-2001/connector-micro-sd-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; Farnell Part Number (none) -> 2614940; Farnell Price (none) -> 1.87; JLC Part Number (none) -> C164170; JLC Price (none) -> 0.43; MPN (none) -> 47219-2001
- J4: JLC Part Number (none) -> N/A; JLC Price (none) -> N/A; MPN (none) -> N/A; now not fitted
- L1: value 1uH -> 3.3uH; Farnell Link (none) -> https://uk.farnell.com/abracon/aota-b201610s3r3-101-t/power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; Farnell Part Number (none) -> 4568814; Farnell Price (none) -> 1.4; JLC Part Number (none) -> C42411119; JLC Price (none) -> 0.14; MPN (none) -> AOTA-B201610S3R3-101-T
- LED1: JLC Part Number (none) -> C12624; JLC Price (none) -> 0.009; MPN (none) -> KT-0603G
- LED2: JLC Part Number (none) -> C2286; JLC Price (none) -> 0.004; MPN (none) -> KT-0603R
- R1, R2: footprint 0_Resistors:R_0402_1005_DensityHigh -> 0_Resistors:R_0603_1608_DensityHigh; JLC Part Number (none) -> C25190; JLC Price (none) -> 0.0008; MPN (none) -> 0603WAF270JT5E
- R10, R9: value 4k7R -> 4.7kR; JLC Part Number (none) -> C23162; JLC Price (none) -> 0.0008; MPN (none) -> 0603WAF4701T5E
- R3: JLC Part Number (none) -> C25105; JLC Price (none) -> 0.0004; MPN (none) -> 0402WGF330JTCE
- R4: JLC Part Number (none) -> C25804; JLC Price (none) -> 0.0007; MPN (none) -> 0603WAF1002T5E
- R5: JLC Part Number (none) -> C21190; JLC Price (none) -> 0.0007; MPN (none) -> 0603WAF1001T5E
- R6: footprint 0_Resistors:R_0402_1005_DensityHigh -> 0_Resistors:R_0603_1608_DensityHigh; JLC Part Number (none) -> C21190; JLC Price (none) -> 0.0007; MPN (none) -> 0603WAF1001T5E
- R7, R8: value ?220R? -> 51R; JLC Part Number (none) -> C23197; JLC Price (none) -> 0.0008; MPN (none) -> 0603WAF510JT5E
- U1: value RP2350_80QFN -> RP2350B; Farnell Link (none) -> https://uk.farnell.com/raspberry-pi/rp2350b-tr7/mcu-32bit-1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; Farnell Part Number (none) -> N/A; Farnell Price (none) -> N/A; JLC Part Number (none) -> C42415655; JLC Price (none) -> 0.89; MPN (none) -> RP2350B
- U2: Farnell Link (none) -> https://uk.farnell.com/infineon/s25fl128lagmfi013/flash-mem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; Farnell Part Number (none) -> 4128033; Farnell Price (none) -> 1.94; JLC Part Number (none) -> C97521; JLC Price (none) -> 1.13; Supplier Link https://uk.farnell.com/infineon/s25fl128lagmfi013/flash-mem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 -> (none)
- X1: Farnell Link (none) -> https://uk.farnell.com/abracon/abm8-272-t3/crystal-12mhz-10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; Farnell Part Number (none) -> 4331750; Farnell Price (none) -> 0.67; JLC Part Number (none) -> C20625731; JLC Price (none) -> 0.25; MPN (none) -> ABM8-272-T3
Connections:
- net PYRO_IN: now also U1.12 (GPIO13); no longer U1.55 (GPIO44_ADC4)
- net SD_DAT1: now also U1.13 (GPIO14); no longer U1.12 (GPIO13)
- net Servo1_PWM: now also U1.57 (GPIO46_ADC6); no longer U1.9 (GPIO11)
- net Servo2_PWM: now also U1.55 (GPIO44_ADC4); no longer U1.11 (GPIO12)
- net Servo3_PWM: now also U1.53 (GPIO42_ADC2); no longer U1.13 (GPIO14)
- net PYRO_SEN: no longer names the net of U1.56 (GPIO45_ADC5)
- net PYRO_SENSE: no longer names the net of U1.54 (GPIO43_ADC3)
- new net PYRO_ST1: U1.11 (GPIO12)
- new net PYRO_ST2: U1.9 (GPIO11)
Other:
- note removed: "1v1 VDD Decoupling"
- note removed: "3v3 VDD Decoupling All 100nF"
- note removed: "4.7uF below VREG"
- note removed: "I2C Pull Ups"
- note removed: "Jumper to program with USB"
- title: Sheet Title A -> MCU & Peripherals
- moved on the sheet: BUZ1, C1, C10, C11, C12, C13, C14, C15, C16, C17, C18, C19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

Commit message: PCBs update - Near Complete x2
Parts:
- added Q1: MMBT5551, 0_Passives:SOT-23, symbol 0_Passives:MMBT5551
- added R9: 1kR, 0_Resistors:R_0402_1005_DensityMedium, symbol 0_Passives:R
- BUZ1: footprint 0_Passives:BUZZER,7.5x7.5mm -> 0_Passives:BUZZER,5x5mm; JLC Part Number C95299 -> (none); JLC Price 0.17 -> (none); MPN MLT-7525 -> KSSG33J12Y; Min Qty (none) -> 5; Order Code (none) -> 4245943; Part Link (none) -> https://uk.farnell.com/kingstate/kssg33j12y/magnetic-transd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; Price Per (none) -> 1.06; Supplier (none) -> Farnell
- C1, C15, C2, C3: JLC Part Number C23733 -> (none); JLC Price 0.0035 -> (none); Min Qty (none) -> 20; Order Code (none) -> C23733; Price Per (none) -> 0.0035; Supplier (none) -> JLCPCB
- C10, C11, C12, C13, C14, C4, C5, C6, C7, C8, C9: JLC Part Number C1525 -> (none); JLC Price 0.0009 -> (none); Min Qty (none) -> 20; Order Code (none) -> C1525; Price Per (none) -> 0.0009; Supplier (none) -> JLCPCB
- C16, C17: JLC Part Number C1548 -> (none); JLC Price 0.0007 -> (none); Min Qty (none) -> 20; Order Code (none) -> C1548; Price Per (none) -> 0.0007; Supplier (none) -> JLCPCB
- C18, C19: JLC Part Number C14663 -> (none); JLC Price 0.002 -> (none); Min Qty (none) -> 20; Order Code (none) -> C14663; Price Per (none) -> 0.002; Supplier (none) -> JLCPCB
- D1: value ~ -> 1N4148WS; JLC Part Number C2128 -> (none); JLC Price 0.0064 -> (none); Min Qty (none) -> 20; Order Code (none) -> C2128; Price Per (none) -> 0.0062; Supplier (none) -> JLCPCB
- J12: Farnell Link https://uk.farnell.com/molex/502352-0201/wtb-conn-header-2p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 -> (none); Farnell Part Number 3103081 -> (none); Farnell Price 0.95 -> (none); JLC Part Number C587898 -> (none); JLC Price 0.22 -> (none); Min Qty (none) -> 1; Order Code (none) -> 3103081; Part Link (none) -> https://uk.farnell.com/molex/502352-0201/wtb-conn-header-2p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; Price Per (none) -> 0.95; Supplier (none) -> Farnell
- J13: symbol Connector_Generic:Conn_02x03_Odd_Even -> 0_Connectors:Conn_02x03_Odd_Even; JLC Part Number N/A -> (none); JLC Price N/A -> (none); now fitted
- J3: Farnell Link https://uk.farnell.com/molex/47219-2001/connector-micro-sd-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 -> (none); Farnell Part Number 2614940 -> (none); Farnell Price 1.87 -> (none); JLC Part Number C164170 -> (none); JLC Price 0.43 -> (none); Min Qty (none) -> 1; Order Code (none) -> 2614940; Part Link (none) -> https://uk.farnell.com/molex/47219-2001/connector-micro-sd-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; Price Per (none) -> 1.87; Supplier (none) -> Farnell
- J4: JLC Part Number N/A -> (none); JLC Price N/A -> (none); now fitted
- L1: Farnell Link https://uk.farnell.com/abracon/aota-b201610s3r3-101-t/power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 -> (none); Farnell Part Number 4568814 -> (none); Farnell Price 1.4 -> (none); JLC Part Number C42411119 -> (none); JLC Price 0.14 -> (none); Min Qty (none) -> 5; Order Code (none) -> C42411119; Price Per (none) -> 0.14; Supplier (none) -> JLCPCB
- LED1: JLC Part Number C12624 -> (none); JLC Price 0.009 -> (none); MPN KT-0603G -> MP008288; Min Qty (none) -> 5; Order Code (none) -> 3796319; Part Link (none) -> https://uk.farnell.com/multicomp-pro/mp008288/led-green-90m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; Price Per (none) -> 0.13; Supplier (none) -> Farnell
- LED2: JLC Part Number C2286 -> (none); JLC Price 0.004 -> (none); MPN KT-0603R -> MP008277; Min Qty (none) -> 5; Order Code (none) -> 3796306; Part Link (none) -> https://uk.farnell.com/multicomp-pro/mp008277/led-red-220mc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; Price Per (none) -> 0.13; Supplier (none) -> Farnell
- R1, R2: JLC Part Number C25190 -> (none); JLC Price 0.0008 -> (none); Min Qty (none) -> 20; Order Code (none) -> C25190; Price Per (none) -> 0.0008; Supplier (none) -> JLCPCB
- R10: renamed from R9; JLC Part Number C23162 -> (none); JLC Price 0.0008 -> (none); Min Qty (none) -> 20; Order Code (none) -> C23162; Price Per (none) -> 0.0008; Supplier (none) -> JLCPCB
- R11: renamed from R10; JLC Part Number C23162 -> (none); JLC Price 0.0008 -> (none); Min Qty (none) -> 20; Order Code (none) -> C23162; Price Per (none) -> 0.0008; Supplier (none) -> JLCPCB
- R3: JLC Part Number C25105 -> (none); JLC Price 0.0004 -> (none); Min Qty (none) -> 20; Order Code (none) -> C25105; Price Per (none) -> 0.0004; Supplier (none) -> JLCPCB
- R4: JLC Part Number C25804 -> (none); JLC Price 0.0007 -> (none); Min Qty (none) -> 20; Order Code (none) -> C25804; Price Per (none) -> 0.0007; Supplier (none) -> JLCPCB
- R5, R6: footprint 0_Resistors:R_0603_1608_DensityHigh -> 0_Resistors:R_0402_1005_DensityMedium; JLC Part Number C21190 -> (none); JLC Price 0.0007 -> (none); MPN 0603WAF1001T5E -> 0402WGF1001TCE; Min Qty (none) -> 20; Order Code (none) -> C11702; Price Per (none) -> 0.0004; Supplier (none) -> JLCPCB
- R7, R8: JLC Part Number C23197 -> (none); JLC Price 0.0008 -> (none); Min Qty (none) -> 20; Order Code (none) -> C23197; Price Per (none) -> 0.0008; Supplier (none) -> JLCPCB
- U1: Farnell Link https://uk.farnell.com/raspberry-pi/rp2350b-tr7/mcu-32bit-1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 -> (none); Farnell Part Number N/A -> (none); Farnell Price N/A -> (none); JLC Part Number C42415655 -> (none); JLC Price 0.89 -> (none); Min Qty (none) -> 1; Order Code (none) -> C42415655; Price Per (none) -> 0.89; Supplier (none) -> JLCPCB
- U2: Farnell Link https://uk.farnell.com/infineon/s25fl128lagmfi013/flash-mem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 -> (none); Farnell Part Number 4128033 -> (none); Farnell Price 1.94 -> (none); JLC Part Number C97521 -> (none); JLC Price 1.13 -> (none); Min Qty (none) -> 1; Order Code (none) -> 4128033; Part Link (none) -> https://uk.farnell.com/infineon/s25fl128lagmfi013/flash-mem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; Price Per (none) -> 1.62; Supplier (none) -> Farnell
- X1: Farnell Link https://uk.farnell.com/abracon/abm8-272-t3/crystal-12mhz-10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 -> (none); Farnell Part Number 4331750 -> (none); Farnell Price 0.67 -> (none); JLC Part Number C20625731 -> (none); JLC Price 0.25 -> (none); Min Qty (none) -> 1; Order Code (none) -> 4331750; Part Link (none) -> https://uk.farnell.com/abracon/abm8-272-t3/crystal-12mhz-10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; Price Per (none) -> 0.67; Supplier (none) -> Farnell
Connections:
- net +3V3: now also BUZ1.1 (+), D1.1 (K)
- net GND: now also Q1.2 (E); no longer BUZ1.3 (GND)
- removed net STATUS_BUZZER+: BUZ1.1 (+), D1.1 (K), U1.45 (GPIO36)
- net STATUS_BUZZER-: no longer names the net of BUZ1.2 (-), D1.2 (A)
- net STATUS_BUZZER-: now also Q1.3 (C); no longer U1.44 (GPIO35)
- new net: Q1.1 (B), R9.2
- new net STATUS_BUZZER: R9.1, U1.45 (GPIO36)
- no-connect marks 21 -> 22
Other:
- moved on the sheet: LED1, LED2, R7, R8
