File: COMET1_CCT_Board/SubSchematics/Sensors.kicad_sch (KiCad schematic)
At the start: 27 parts, among them J10 Molex_01x02, J11 Molex_01x02, J7 Molex_01x02, J8 Molex_01x02, J9 Molex_01x02, U5 LM27313XMFX_NOPB, U6 PAC1934T-I_JQ, U7 MCP96RL00-E_MX, U8 MCP96RL00-E_MX, U9 STS4L-AD1B-R3

Commit message: PCBs Update - Near Complete
Parts:
- C25, C26: JLC Part Number (none) -> C19666; JLC Price (none) -> 0.007; MPN (none) -> CL10A475KO8NNNC
- C27, C28, C30, C32, C33: JLC Part Number (none) -> C14663; JLC Price (none) -> 0.002; MPN (none) -> CC0603KRX7R9BB104
- C29, C31: JLC Part Number (none) -> C57112; JLC Price (none) -> 0.002; MPN (none) -> 0603B103K500NT
- D3: footprint 0_Passives:D_0805_2012Metric -> 0_Passives:D_SOD-123; JLC Part Number (none) -> C8598; JLC Price (none) -> 0.017; MPN (none) -> B5819W SL
- J10, J11, J7, J8, J9: Farnell Link (none) -> https://uk.farnell.com/molex/502352-0201/wtb-conn-header-2p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; Farnell Part Number (none) -> 3103081; Farnell Price (none) -> 0.95; JLC Part Number (none) -> C587898; JLC Price (none) -> 0.22; Supplier Link https://uk.farnell.com/molex/502352-0201/wtb-conn-header-2p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 -> (none)
- L2: JLC Part Number (none) -> C1051; JLC Price (none) -> 0.015; MPN (none) -> CMI321609X100KT
- R17, R18, R19: value 0R2 -> 0.1R; JLC Part Number (none) -> C25334; JLC Price (none) -> 0.0037; MPN (none) -> 1206W4F100LT5E
- R20: value 118kR -> 120kR; JLC Part Number (none) -> C25808; JLC Price (none) -> 0.0008; MPN (none) -> 0603WAF1203T5E
- R21: value 13.3kR -> 13kR; JLC Part Number (none) -> C22797; JLC Price (none) -> 0.0008; MPN (none) -> 0603WAF1302T5E
- R22: footprint 0_Resistors:R_0805_2012_DensityHigh -> 0_Resistors:R_0603_1608_DensityHigh; JLC Part Number (none) -> N/A; JLC Price (none) -> N/A; MPN (none) -> N/A; now not fitted
- U5: value LM27313XMFX_NOPB -> LM27313; footprint 0_Power:SOT95P280X145-5N -> 0_Power:SOT-23-5; Farnell Link (none) -> https://uk.farnell.com/texas-instruments/lm27313xmfx-nopb/d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; Farnell Part Number (none) -> 3121547; Farnell Price (none) -> 1.85; JLC Part Number (none) -> C341750; JLC Price (none) -> 0.32; Supplier Link https://uk.farnell.com/texas-instruments/lm27313xmfx-nopb/d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 -> (none)
- U6: value PAC1934T-I_JQ -> PAC1934; footprint 0_Sensors:QFN65P400X400X55-17N-D -> 0_Sensors:PAC1934T-I_JQ; Farnell Link (none) -> https://uk.farnell.com/microchip/pac1934t-i-jq/dc-power-ene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; Farnell Part Number (none) -> 2907898; Farnell Price (none) -> 1.72; Height 0.55 -> (none); JLC Part Number (none) -> C623960; JLC Price (none) -> 2.03; MPN (none) -> PAC1934T-I/JQ; Manufacturer_Name Microchip -> (none); Manufacturer_Part_Number PAC1934T-I/JQ -> (none)
- U7, U8: value MCP96RL00-E_MX -> MCP96R00; footprint 0_Sensors:QFN65P500X500X100-21N-D -> 0_Sensors:MCP9600L00; Farnell Link (none) -> https://uk.farnell.com/microchip/mcp96rl00-e-mx/thermocoupl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; Farnell Part Number (none) -> 2991624; Farnell Price (none) -> 3.49; Height 1 -> (none); JLC Part Number (none) -> C638823; JLC Price (none) -> 4.57; Manufacturer_Name Microchip -> (none); Manufacturer_Part_Number MCP96RL00-E/MX -> (none); Supplier Link https://uk.farnell.com/microchip/mcp96rl00-e-mx/thermocoupl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 -> (none)
- U9: value STS4L-AD1B-R3 -> STS4x; Farnell Link (none) -> https://uk.farnell.com/sensirion/sts4l-ad1b-r3/temperature-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; Farnell Part Number (none) -> 4551122; Farnell Price (none) -> 0.52; JLC Part Number (none) -> C3663715; JLC Price (none) -> 0.38; Supplier Link https://uk.farnell.com/sensirion/sts4l-ad1b-r3/temperature-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 -> (none)
Other:
- title: Sheet Title A -> Sensors

Commit message: PCBs update - Near Complete x2
Parts:
- removed R22: 0R, 0_Resistors:R_0603_1608_DensityHigh, symbol 0_Passives:R
- C25, C26: JLC Part Number C19666 -> (none); JLC Price 0.007 -> (none); Min Qty (none) -> 20; Order Code (none) -> C19666; Price Per (none) -> 0.007; Supplier (none) -> JLCPCB
- C27, C28, C30, C32, C33: JLC Part Number C14663 -> (none); JLC Price 0.002 -> (none); Min Qty (none) -> 20; Order Code (none) -> C14663; Price Per (none) -> 0.002; Supplier (none) -> JLCPCB
- C29, C31: value 10nF -> 100nF; JLC Part Number C57112 -> (none); JLC Price 0.002 -> (none); MPN 0603B103K500NT -> CC0603KRX7R9BB104; Min Qty (none) -> 20; Order Code (none) -> C14663; Price Per (none) -> 0.002; Supplier (none) -> JLCPCB
- D3: JLC Part Number C8598 -> (none); JLC Price 0.017 -> (none); Min Qty (none) -> 20; Order Code (none) -> C8598; Price Per (none) -> 0.017; Supplier (none) -> JLCPCB
- J10, J11, J7, J8, J9: Farnell Link https://uk.farnell.com/molex/502352-0201/wtb-conn-header-2p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 -> (none); Farnell Part Number 3103081 -> (none); Farnell Price 0.95 -> (none); JLC Part Number C587898 -> (none); JLC Price 0.22 -> (none); Min Qty (none) -> 1; Order Code (none) -> 3103081; Part Link (none) -> https://uk.farnell.com/molex/502352-0201/wtb-conn-header-2p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; Price Per (none) -> 0.95; Supplier (none) -> Farnell
- L2: JLC Part Number C1051 -> (none); JLC Price 0.015 -> (none); MPN CMI321609X100KT -> MCSD54-120MU; Min Qty (none) -> 1; Order Code (none) -> 1864116; Part Link (none) -> https://uk.farnell.com/multicomp-pro/mcsd54-120mu/inductor-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; Price Per (none) -> 0.25; Supplier (none) -> Farnell
- R18: renamed from R17; JLC Part Number C25334 -> (none); JLC Price 0.0037 -> (none); Min Qty (none) -> 15; Order Code (none) -> C25334; Price Per (none) -> 0.0037; Supplier (none) -> JLCPCB
- R19: renamed from R18; JLC Part Number C25334 -> (none); JLC Price 0.0037 -> (none); Min Qty (none) -> 15; Order Code (none) -> C25334; Price Per (none) -> 0.0037; Supplier (none) -> JLCPCB
- R20: renamed from R19; JLC Part Number C25334 -> (none); JLC Price 0.0037 -> (none); Min Qty (none) -> 15; Order Code (none) -> C25334; Price Per (none) -> 0.0037; Supplier (none) -> JLCPCB
- R21: renamed from R20; JLC Part Number C25808 -> (none); JLC Price 0.0008 -> (none); Min Qty (none) -> 20; Order Code (none) -> C25808; Price Per (none) -> 0.0008; Supplier (none) -> JLCPCB
- R22: renamed from R21; JLC Part Number C22797 -> (none); JLC Price 0.0008 -> (none); Min Qty (none) -> 20; Order Code (none) -> C22797; Price Per (none) -> 0.0008; Supplier (none) -> JLCPCB
- U5: Farnell Link https://uk.farnell.com/texas-instruments/lm27313xmfx-nopb/d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 -> (none); Farnell Part Number 3121547 -> (none); Farnell Price 1.85 -> (none); JLC Part Number C341750 -> (none); JLC Price 0.32 -> (none); Min Qty (none) -> 1; Order Code (none) -> 3121547; Part Link (none) -> https://uk.farnell.com/texas-instruments/lm27313xmfx-nopb/d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; Price Per (none) -> 1.85; Supplier (none) -> Farnell
- U6: Farnell Link https://uk.farnell.com/microchip/pac1934t-i-jq/dc-power-ene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 -> (none); Farnell Part Number 2907898 -> (none); Farnell Price 1.72 -> (none); JLC Part Number C623960 -> (none); JLC Price 2.03 -> (none); Min Qty (none) -> 1; Order Code (none) -> 2907898; Part Link (none) -> https://uk.farnell.com/microchip/pac1934t-i-jq/dc-power-ene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; Price Per (none) -> 1.72; Supplier (none) -> Farnell
- U7, U8: Farnell Link https://uk.farnell.com/microchip/mcp96rl00-e-mx/thermocoupl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 -> (none); Farnell Part Number 2991624 -> (none); Farnell Price 3.49 -> (none); JLC Part Number C638823 -> (none); JLC Price 4.57 -> (none); Min Qty (none) -> 1; Order Code (none) -> 2991624; Part Link (none) -> https://uk.farnell.com/microchip/mcp96rl00-e-mx/thermocoupl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; Price Per (none) -> 3.49; Supplier (none) -> Farnell
- U9: value STS4x -> STS4L; Farnell Link https://uk.farnell.com/sensirion/sts4l-ad1b-r3/temperature-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 -> (none); Farnell Part Number 4551122 -> (none); Farnell Price 0.52 -> (none); JLC Part Number C3663715 -> (none); JLC Price 0.38 -> (none); Min Qty (none) -> 1; Order Code (none) -> 4551122; Part Link (none) -> https://uk.farnell.com/sensirion/sts4l-ad1b-r3/temperature-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; Price Per (none) -> 0.52; Supplier (none) -> Farnell
Connections:
- net GND: now also U6.6 (ADDRSEL)
Other:
- note added: "I2C - 0x20"
- note added: "I2C - 0x44"
- note added: "I2C - 0x60"
- note added: "I2C - 0x6E"
- note removed: "I2C Address: 0x40"
- note removed: "Potential I2C Addresses: 0x44, 0x45, 0x46"
- moved on the sheet: C30, C32
