File: COMET1_PWR_Board/SubSchematics/PowerBoard.kicad_sch (KiCad schematic)
At the start: 40 parts, among them J1 XT30_THT_H, J2 Molex_Block_01x02, J3 502352-0301, J4 502352-0301, J5 502352-0301, J6 DF11-10DP-2DSA, J7 DF11-10DP-2DSA, U1 NCP1117_3.3, U2 BV1HJ180EFJ-C, U3 MIC29302AWD, U4 MIC29302AWD

Commit message: PCBs update - Near Complete x2
Parts:
- C1, C2: JLC_MPN 0603B103K500NT -> (none); JLC_PART C57112 -> (none); MPN (none) -> 0603B103K500NT; Min Qty (none) -> 20; Order Code (none) -> C57112; Price Per (none) -> 0.002; Supplier (none) -> JLCPCB
- C3: JLC_MPN CC0603KRX7R9BB104 -> (none); JLC_PART C14663 -> (none); MPN (none) -> CC0603KRX7R9BB104; Min Qty (none) -> 20; Order Code (none) -> C14663; Price Per (none) -> 0.002; Supplier (none) -> JLCPCB
- C4, C5, C6, C7: JLC_MPN CL10A106KP8NNNC -> (none); JLC_PART C19702 -> (none); MPN (none) -> CL10A106KP8NNNC; Min Qty (none) -> 20; Order Code (none) -> C19702; Price Per (none) -> 0.002; Supplier (none) -> JLCPCB
- F1, F2: JLC_MPN SMD1210B075TF/24 -> (none); JLC_PART C634245 -> (none); Min Qty (none) -> 5; Order Code (none) -> 4072044; Price Per (none) -> 0.12; Supplier (none) -> Farnell
- J1: JLC_MPN XT30PW-M30.G.Y -> (none); JLC_PART C431092 -> (none); Manufacturer_Name Multicomp Pro -> (none); Min Qty (none) -> 5; Order Code (none) -> 4220281; Price Per (none) -> 0.39; Supplier (none) -> Farnell
- J2: JLC_MPN 2060-452/998-404 -> (none); JLC_PART C2765055 -> (none); Min Qty (none) -> 1; Order Code (none) -> 2499130; Price Per (none) -> 0.76; Supplier (none) -> Farnell
- J3, J4, J5: JLC_MPN 5023520301 -> (none); JLC_PART C587901 -> (none); Min Qty (none) -> 10; Order Code (none) -> 3365016; Price Per (none) -> 0.84; Supplier (none) -> Farnell
- J6, J7: JLC_MPN DF11-10DP-2DSA(08) -> (none); JLC_PART C506656 -> (none); Manufacturer_Name Hirose -> (none); Min Qty (none) -> 10; Order Code (none) -> 1688345; Price Per (none) -> 0.6; Supplier (none) -> Farnell
- LED1: JLC_MPN KT-0603R -> (none); JLC_PART C2286 -> (none); MPN (none) -> MP008277; Min Qty (none) -> 5; Order Code (none) -> 3796306; Price Per (none) -> 0.13; Supplier (none) -> Farnell
- R1: JLC_MPN 0603WAF4703T5E -> (none); JLC_PART C23178 -> (none); MPN (none) -> 0603WAF4703T5E; Min Qty (none) -> 20; Order Code (none) -> C23178; Price Per (none) -> 0.0008; Supplier (none) -> JLCPCB
- R10, R11: JLC_MPN 0603WAF1002T5E -> (none); JLC_PART C25804 -> (none); MPN (none) -> 0603WAF1002T5E; Min Qty (none) -> 20; Order Code (none) -> C25804; Price Per (none) -> 0.0008; Supplier (none) -> JLCPCB
- R12: JLC_MPN 0603WAF5102T5E -> (none); JLC_PART C23196 -> (none); MPN (none) -> 0603WAF5102T5E; Min Qty (none) -> 20; Order Code (none) -> C23196; Price Per (none) -> 0.0008; Supplier (none) -> JLCPCB
- R2: JLC_MPN 0603WAF3903T5E -> (none); JLC_PART C23150 -> (none); MPN (none) -> 0603WAF3903T5E; Min Qty (none) -> 20; Order Code (none) -> C23150; Price Per (none) -> 0.0008; Supplier (none) -> JLCPCB
- R3: JLC_MPN 0603WAF510JT5E -> (none); JLC_PART C23197 -> (none); MPN (none) -> 0603WAF510JT5E; Min Qty (none) -> 20; Order Code (none) -> C23197; Price Per (none) -> 0.0008; Supplier (none) -> JLCPCB
- R5: JLC_MPN 0603WAF4701T5E -> (none); JLC_PART C23162 -> (none); MPN (none) -> 0603WAF4701T5E; Min Qty (none) -> 20; Order Code (none) -> C23162; Price Per (none) -> 0.0008; Supplier (none) -> JLCPCB
- R6, R8: JLC_MPN 0603WAF4700T5E -> (none); JLC_PART C23179 -> (none); MPN (none) -> 0603WAF4700T5E; Min Qty (none) -> 20; Order Code (none) -> C23179; Price Per (none) -> 0.0008; Supplier (none) -> JLCPCB
- R7, R9: JLC_MPN 0603WAF1200T5E -> (none); JLC_PART C22787 -> (none); MPN (none) -> 0603WAF1200T5E; Min Qty (none) -> 20; Order Code (none) -> C22787; Price Per (none) -> 0.0008; Supplier (none) -> JLCPCB
- S1: JLC_MPN SS-12D06-G030 -> (none); JLC_PART C17179519 -> (none); MPN 1101M2S3AQE2 -> (none); Supplier (none) -> Farnell
- U1: JLC_MPN NCP1117LPST33T3G -> (none); JLC_PART C146799 -> (none); Min Qty (none) -> 5; Order Code (none) -> 2534283; Price Per (none) -> 1.91; Supplier (none) -> Farnell
- U2: JLC_MPN BV1HJ180EFJ-CE2 -> (none); JLC_PART C17347420 -> (none); Min Qty (none) -> 1; Order Code (none) -> 4137626; Price Per (none) -> 0.96; Supplier (none) -> Farnell; Supplier Link (none) -> https://uk.farnell.com/rohm/bv1hj180efj-ce2/power-load-sw-h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; Supplier_Link https://uk.farnell.com/rohm/bv1hj180efj-ce2/power-load-sw-h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 -> (none)
- U3, U4: JLC_MPN MIC29302AWD-TR -> (none); JLC_PART C627907 -> (none); Min Qty (none) -> 1; Order Code (none) -> 2857615; Price Per (none) -> 2.28; Supplier (none) -> Farnell; Supplier Link (none) -> https://uk.farnell.com/microchip/mic29302awd-tr/ldo-adj-1-2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; Supplier_Link https://uk.farnell.com/microchip/mic29302awd-tr/ldo-adj-1-2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 -> (none)
